File: half_qwerty.kicad_pcb (KiCad board)
At the start: 2 copper layers, 142.9 x 81.9 mm, 71 parts, among them J1 USB_C_Receptacle_USB2.0, SW1 SW_Push, SW10 SW_Push, SW11 SW_Push, SW12 SW_Push, SW13 SW_Push, SW14 SW_Push, SW15 SW_Push, SW16 SW_Push, SW17 SW_Push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

Commit message: done for now
Parts:
- added D25: LED, LED_SMD:LED_0805_2012Metric_Pad1.15x1.40mm_HandSolder, F.Cu at (167.4, 133.3)
- added D26: LED, LED_SMD:LED_0805_2012Metric_Pad1.15x1.40mm_HandSolder, F.Cu at (167.4, 138.1)
- added D27: LED, LED_SMD:LED_0805_2012Metric_Pad1.15x1.40mm_HandSolder, F.Cu at (167.4, 142.9)
- added R10: 1k, Resistor_SMD:R_0603_1608Metric_Pad1.05x0.95mm_HandSolder, F.Cu at (171.2, 140.5)
- added R8: 1k, Resistor_SMD:R_0603_1608Metric_Pad1.05x0.95mm_HandSolder, F.Cu at (171.2, 131.6)
- added R9: 1k, Resistor_SMD:R_0603_1608Metric_Pad1.05x0.95mm_HandSolder, F.Cu at (171.2, 133.3)
- moved R5 3.07 mm to (168.7, 140.5), turned to 315 degrees
- moved D15 1.63 mm to (215.4, 85.6), turned to 90 degrees
Connections:
- D1 pad 1: /row0 -> /PD4
- D11 pad 1: /row2 -> /PF6
- D12 pad 1: /row2 -> /PF6
- D13 pad 1: /row2 -> /PF6
- D14 pad 1: /row2 -> /PF6
- D15 pad 1: /row2 -> /PF6
- D16 pad 1: /row3 -> /PF7
- D17 pad 1: /row3 -> /PF7
- D18 pad 1: /row3 -> /PF7
- D19 pad 1: /row3 -> /PF7
- D2 pad 1: /row0 -> /PD4
- D20 pad 1: /row3 -> /PF7
- D21 pad 1: /row4 -> /PB6
- D22 pad 1: /row4 -> /PB6
- D3 pad 1: /row0 -> /PD4
- D4 pad 1: /row0 -> /PD4
- D5 pad 1: /row0 -> /PD4
- SW1 pad 1: /col0 -> /PF4
- SW10 pad 1: /col4 -> /PD7
- SW11 pad 1: /col0 -> /PF4
- SW12 pad 1: /col1 -> /PF1
- SW13 pad 1: /col2 -> /PF5
- SW14 pad 1: /col3 -> /PB7
- SW15 pad 1: /col4 -> /PD7
- SW16 pad 1: /col0 -> /PF4
- SW17 pad 1: /col1 -> /PF1
- SW18 pad 1: /col2 -> /PF5
- SW19 pad 1: /col3 -> /PB7
- SW2 pad 1: /col1 -> /PF1
- SW20 pad 1: /col4 -> /PD7
- SW21 pad 1: /col3 -> /PB7
- SW22 pad 1: /col4 -> /PD7
- SW3 pad 1: /col2 -> /PF5
- SW4 pad 1: /col3 -> /PB7
- SW5 pad 1: /col4 -> /PD7
- SW6 pad 1: /col0 -> /PF4
- SW7 pad 1: /col1 -> /PF1
- SW8 pad 1: /col2 -> /PF5
- SW9 pad 1: /col3 -> /PB7
Routing:
- net /PF6: track 0.00 -> 156.3 mm, vias 0 -> 6
- net /PF4: track 0.00 -> 153.7 mm, vias 0 -> 2
- net /PD4: track 0.00 -> 148.5 mm, vias 0 -> 6
- net /PD7: track 0.00 -> 147.8 mm, vias 0 -> 7
- net /PF7: track 0.00 -> 140.5 mm, vias 0 -> 8
- net /PB7: track 0.00 -> 140.5 mm, vias 0 -> 10
- net /PF1: track 0.00 -> 122.3 mm, vias 0 -> 10
- net /PF5: track 0.00 -> 119.0 mm, vias 0 -> 6
- net /row0: track 81.7 -> 0.00 mm
- net /PB6: track 0.00 -> 74.8 mm, vias 0 -> 6
- net /col0: track 68.9 -> 0.00 mm
- net /row2: track 66.9 -> 0.00 mm
- net /row3: track 58.7 -> 0.00 mm
- net /col3: track 46.8 -> 0.00 mm, vias 4 -> 0
- net /row4: track 25.5 -> 0.00 mm
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Other:
- board text added: "(optional)"
