File: half_qwerty.kicad_pcb (KiCad board)
At the start: 2 copper layers, 142.9 x 81.9 mm, 77 parts, among them J1 USB_C_Receptacle_USB2.0, SW1 SW_Push, SW10 SW_Push, SW11 SW_Push, SW12 SW_Push, SW13 SW_Push, SW14 SW_Push, SW15 SW_Push, SW16 SW_Push, SW17 SW_Push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

Commit message: recheck and var. alpha ordered
Parts:
- added G***: LOGO, a40:keyaki_namiki-icon, F.Cu at (208.8, 136.9)
- J1: moved to F.Cu
- moved R7 3.87 mm to (200.3, 74.2), turned to 180 degrees
- moved R6 2.62 mm to (195.0, 75.9), turned to 0 degrees
- moved R4 0.77 mm to (195.0, 74.2)
- moved J1 0.14 mm to (197.5, 65.8), turned to 180 degrees
Connections:
- D10 pad 1: /row1 -> /PF0
- D6 pad 1: /row1 -> /PF0
- D7 pad 1: /row1 -> /PF0
- D8 pad 1: /row1 -> /PF0
- D9 pad 1: /row1 -> /PF0
Routing:
- net /PF0: track 0.00 -> 141.6 mm, vias 0 -> 6
- net /row1: track 101.4 -> 0.00 mm
- net /CC2: track 7.87 -> 13.3 mm, vias 2 -> 0
- net GND: track 288.0 -> 283.5 mm, vias 17 -> 15
- net /PB6: track 74.8 -> 76.2 mm
- net /PF4: track 153.7 -> 154.8 mm
- net /CC1: track 6.56 -> 7.54 mm
- net Net-(J1-PadS1): track 20.3 -> 19.4 mm
- net /PB7: track 140.5 -> 141.4 mm
- net /RESET: track 37.0 -> 36.2 mm
- net /PD7: track 147.8 -> 148.4 mm
Other:
- board text removed: "(optional)"
