File: half_qwerty.sch (KiCad schematic (older format))
At the start: 71 parts, among them J1 USB_C_Receptacle_USB2.0, SW1 SW_Push, SW10 SW_Push, SW11 SW_Push, SW12 SW_Push, SW13 SW_Push, SW14 SW_Push, SW15 SW_Push, SW16 SW_Push, SW17 SW_Push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

Commit message: done for now
Parts:
- added D25, D26, D27: LED, LED_SMD:LED_0805_2012Metric_Pad1.15x1.40mm_HandSolder, symbol Device:LED
- added R10, R8, R9: 1k, Resistor_SMD:R_0603_1608Metric_Pad1.05x0.95mm_HandSolder, symbol Device:R
- SW23: footprint Button_Switch_SMD:Panasonic_EVQPUL_EVQPUC -> Button_Switch_SMD:SW_SPST_TL3342
Connections:
- net col0 is gone; now on net PF4: SW1.1, SW11.1, SW16.1, SW6.1
- net col1 is gone; now on net PF1: SW12.1, SW17.1, SW2.1, SW7.1
- net col2 is gone; now on net PF5: SW13.1, SW18.1, SW3.1, SW8.1
- net col3 is gone; now on net PB7: SW14.1, SW19.1, SW21.1, SW4.1, SW9.1
- net col4 is gone; now on net PD7: SW10.1, SW15.1, SW20.1, SW22.1, SW5.1
- net row0 is gone; now on net PD4: D1.1 (K), D2.1 (K), D3.1 (K), D4.1 (K), D5.1 (K)
- net row2 is gone; now on net PF6: D11.1 (K), D12.1 (K), D13.1 (K), D14.1 (K), D15.1 (K)
- net row3 is gone; now on net PF7: D16.1 (K), D17.1 (K), D18.1 (K), D19.1 (K), D20.1 (K)
- net row4 is gone; now on net PB6: D21.1 (K), D22.1 (K)
- net GND: now also D25.1 (K), D26.1 (K), D27.1 (K)
- net PB5: now also R10.1
- net PC6: now also R8.1
- net PC7: now also R9.1
- new net: D25.2 (A), R8.2
- new net: D26.2 (A), R9.2
- new net: D27.2 (A), R10.2
Changed lines of the file:
@@
 	0    -1   -1   0
 $EndComp
-Text Label 6350 1800 0    50   ~ 0
-row0
 Text Label 6350 2450 0    50   ~ 0
 row1
-Text Label 6350 3100 0    50   ~ 0
-row2
-Text Label 6350 3750 0    50   ~ 0
-row3
-Text Label 6350 4400 0    50   ~ 0
-row4
-Text Label 6850 800  3    50   ~ 0
-col0
-Text Label 7750 800  3    50   ~ 0
-col1
-Text Label 8650 800  3    50   ~ 0
-col2
-Text Label 9550 800  3    50   ~ 0
-col3
-Text Label 10450 800  3    50   ~ 0
-col4
 Wire Wire Line
 	6850 800  6850 1500
@@
 F 0 "SW23" H 1300 4885 50  0000 C CNN
 F 1 "SW_Push" H 1300 4794 50  0000 C CNN
-F 2 "Button_Switch_SMD:Panasonic_EVQPUL_EVQPUC" H 1300 4800 50  0001 C CNN
+F 2 "Button_Switch_SMD:SW_SPST_TL3342" H 1300 4800 50  0001 C CNN
 F 3 "~" H 1300 4800 50  0001 C CNN
 	1    1300 4600
@@
 	1    0    0    -1
 $EndComp
+Text Label 6350 3750 0    50   ~ 0
+PF7
+Text Label 9550 800  3    50   ~ 0
+PB7
+Text Label 6350 3100 0    50   ~ 0
+PF6
+Text Label 10450 800  3    50   ~ 0
+PD7
+Text Label 6350 1800 0    50   ~ 0
+PD4
+Text Label 8650 800  3    50   ~ 0
+PF5
+Text Label 6350 4400 0    50   ~ 0
+PB6
+$Comp
+L Device:LED D25
+U 1 1 5E8980FE
+P 5700 6900
+F 0 "D25" V 5739 6782 50  0000 R CNN
+F 1 "LED" V 5648 6782 50  0000 R CNN
+F 2 "LED_SMD:LED_0805_2012Metric_Pad1.15x1.40mm_HandSolder" H 5700 6900 50  0001 C CNN
+F 3 "~" H 5700 6900 50  0001 C CNN
+	1    5700 6900
+	0    -1   -1   0
+$EndComp
+Text Label 6850 800  3    50   ~ 0
+PF4
+Text Label 7750 800  3    50   ~ 0
+PF1
+$Comp
+L Device:LED D26
+U 1 1 5E8E6109
+P 6050 6900
+F 0 "D26" V 6089 6782 50  0000 R CNN
+F 1 "LED" V 5998 6782 50  0000 R CNN
+F 2 "LED_SMD:LED_0805_2012Metric_Pad1.15x1.40mm_HandSolder" H 6050 6900 50  0001 C CNN
+F 3 "~" H 6050 6900 50  0001 C CNN
+	1    6050 6900
+	0    -1   -1   0
+$EndComp
+$Comp
+L Device:LED D27
+U 1 1 5E8E6540
+P 6400 6900
+F 0 "D27" V 6439 6782 50  0000 R CNN
+F 1 "LED" V 6348 6782 50  0000 R CNN
+F 2 "LED_SMD:LED_0805_2012Metric_Pad1.15x1.40mm_HandSolder" H 6400 6900 50  0001 C CNN
+F 3 "~" H 6400 6900 50  0001 C CNN
+	1    6400 6900
+	0    -1   -1   0
+$EndComp
+$Comp
+L Device:R R8
+U 1 1 5E8E71F4
+P 5700 6450
+F 0 "R8" H 5770 6496 50  0000 L CNN
+F 1 "1k" H 5770 6405 50  0000 L CNN
+F 2 "Resistor_SMD:R_0603_1608Metric_Pad1.05x0.95mm_HandSolder" V 5630 6450 50  0001 C CNN
+F 3 "~" H 5700 6450 50  0001 C CNN
+	1    5700 6450
+	1    0    0    -1
+$EndComp
+$Comp
+L Device:R R9
+U 1 1 5E8E7CF4
+P 6050 6450
+F 0 "R9" H 6120 6496 50  0000 L CNN
+F 1 "1k" H 6120 6405 50  0000 L CNN
+F 2 "Resistor_SMD:R_0603_1608Metric_Pad1.05x0.95mm_HandSolder" V 5980 6450 50  0001 C CNN
+F 3 "~" H 6050 6450 50  0001 C CNN
+	1    6050 6450
+	1    0    0    -1
+$EndComp
+$Comp
+L Device:R R10
+U 1 1 5E8E809E
+P 6400 6450
+F 0 "R10" H 6470 6496 50  0000 L CNN
+F 1 "1k" H 6470 6405 50  0000 L CNN
+F 2 "Resistor_SMD:R_0603_1608Metric_Pad1.05x0.95mm_HandSolder" V 6330 6450 50  0001 C CNN
+F 3 "~" H 6400 6450 50  0001 C CNN
+	1    6400 6450
+	1    0    0    -1
+$EndComp
+Wire Wire Line
+	6400 6600 6400 6750
+Wire Wire Line
+	6050 6600 6050 6750
+Wire Wire Line
+	5700 6600 5700 6750
+Wire Wire Line
+	5700 7050 5700 7350
+Wire Wire Line
+	6050 7050 6050 7350
+Wire Wire Line
+	6400 7050 6400 7350
+$Comp
+L power:GND #PWR0107
+U 1 1 5E919BAF
+P 5700 7350
+F 0 "#PWR0107" H 5700 7100 50  0001 C CNN
+F 1 "GND" H 5705 7177 50  0000 C CNN
+F 2 "" H 5700 7350 50  0001 C CNN
+F 3 "" H 5700 7350 50  0001 C CNN
+	1    5700 7350
+	1    0    0    -1
+$EndComp
+$Comp
+L power:GND #PWR0108
+U 1 1 5E919F2B
+P 6050 7350
+F 0 "#PWR0108" H 6050 7100 50  0001 C CNN
+F 1 "GND" H 6055 7177 50  0000 C CNN
+F 2 "" H 6050 7350 50  0001 C CNN
+F 3 "" H 6050 7350 50  0001 C CNN
+	1    6050 7350
+	1    0    0    -1
+$EndComp
+$Comp
+L power:GND #PWR0109
+U 1 1 5E91A270
+P 6400 7350
+F 0 "#PWR0109" H 6400 7100 50  0001 C CNN
+F 1 "GND" H 6405 7177 50  0000 C CNN
+F 2 "" H 6400 7350 50  0001 C CNN
+F 3 "" H 6400 7350 50  0001 C CNN
+	1    6400 7350
+	1    0    0    -1
+$EndComp
+Wire Wire Line
+	5700 6300 5700 5950
+Wire Wire Line
+	6050 5950 6050 6300
+Wire Wire Line
+	6400 5950 6400 6300
+Text Label 6050 5950 3    50   ~ 0
+PC7
+Text Label 5700 5950 3    50   ~ 0
+PC6
+Text Label 6400 5950 3    50   ~ 0
+PB5
 $EndSCHEMATC

Commit message: recheck and var. alpha ordered
Connections:
- net row1 is gone; now on net PF0: D10.1 (K), D6.1 (K), D7.1 (K), D8.1 (K), D9.1 (K)
Changed lines of the file:
@@
 	0    -1   -1   0
 $EndComp
-Text Label 6350 2450 0    50   ~ 0
-row1
 Wire Wire Line
 	6850 800  6850 1500
@@
 Text Label 6400 5950 3    50   ~ 0
 PB5
+Text Label 6350 2450 0    50   ~ 0
+PF0
 $EndSCHEMATC
